File: Hardware/QwiicHUD.sch (EAGLE design)
At the start: 25 parts, among them J4 WISECHIP_HUD_FPC

Commit message: x02
Added 12V boost circuit
Parts:
- removed C7: 2.2uF, SparkFun-Capacitors:2.2UF-0603-10V-20%
- removed R3: 8.2k, SparkFun-Resistors:8.2KOHM-0603-1/10W-5%
- added C10: 1.0uF, SparkFun-Capacitors:1.0UF-0603-16V-10%
- added C11: 1.0uF/25V, SparkFun-Capacitors:1.0UF-0805-25V-(+80/-20%)
- added D2: 1A/23V/620mV, SparkFun-DiscreteSemi:DIODE-SCHOTTKY-BAT20J
- added L1: 10uH, 1.81_Greyscale_OLED_Breakout:INDUCTORINDUCTOR_10UH
- added R6: 47k, SparkFun-Resistors:47KOHM-0603-1/10W-1%
- added R7: 5.6k, SparkFun-Resistors:5.6KOHM-0603-1/10W-1%
- added U1: AP3012, 1.81_Greyscale_OLED_Breakout:AP3012
- R2, R4: value 4.7k -> 2.2k; device SparkFun-Resistors:4.7KOHM-0603-1/10W-1% -> SparkFun-Resistors:2.2KOHM-0603-1/10W-1%
Connections:
- net RST renamed !RST
- removed net VCC: C7.1, C8.2, C9.1, J4.VCC, R3.1
- new net 12V: C11.1, C8.2, C9.1, D2.C, J4.VCC, R6.2
- new net N$4: D2.A, L1.2, U1.SW
- new net N$5: R6.1, R7.2, U1.FB
- net 3.3V: now also C10.1, L1.1, U1.!SHDN!, U1.VIN; no longer R3.2
- net GND: now also C10.2, C11.2, R7.1, U1.GND; no longer C7.2
Other:
- note added: "12V Boost"
- note added: "VCC = 1.25 (1 + R1 / R2) = 1.25 (1+ 47/5.6) = 11.74 V"
- note removed: "time constant 1.8ms Tpdr2 = 2ms"
- moved on the sheet: C1, C2, C3, C4, C5, C6, C8, C9, D1, JP1, R1, R2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
