File: Hardware/QwiicHUD.sch (EAGLE design)
At the start: 30 parts, among them J4 WISECHIP_HUD_FPC, U1 AP3012

Commit message: Revert "Changed inductor to inventory part"
This reverts commit 6ab7a03f3320a090153a192dfaf0fd3f0c8c93f1.
Parts:
- L1: device SparkFun-Coils:INDUCTOR-CDRH-10UH -> 1.81_Greyscale_OLED_Breakout:INDUCTORINDUCTOR_10UH
Changed lines of the file:
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@@
 <?xml version="1.0" encoding="utf-8"?>
 <!DOCTYPE eagle SYSTEM "eagle.dtd">
-<eagle version="9.1.3">
+<eagle version="7.7.0">
 <drawing>
 <settings>
 <setting alwaysvectorfont="yes"/>
-<setting keepoldvectorfont="yes"/>
 <setting verticaltext="up"/>
 </settings>
@@
 <part name="R7" library="SparkFun-Resistors" deviceset="5.6KOHM" device="-0603-1/10W-1%" value="5.6k"/>
 <part name="D2" library="SparkFun-DiscreteSemi" deviceset="DIODE-SCHOTTKY" device="-BAT20J" value="1A/23V/620mV"/>
-<part name="L1" library="SparkFun-Coils" deviceset="INDUCTOR" device="-CDRH-10UH" value="10uH"/>
+<part name="L1" library="1.81_Greyscale_OLED_Breakout" deviceset="INDUCTOR" device="INDUCTOR_10UH" value="10uH"/>
 <part name="GND8" library="SparkFun-PowerSymbols" deviceset="GND" device=""/>
 <part name="GND9" library="SparkFun-PowerSymbols" deviceset="GND" device=""/>
